File: LE4/Team1_LE4-2/Team1_LE4-2.kicad_sch (KiCad schematic)
At the start: 24 parts, among them SW1 SW_Push, U1 8086_Min_Mode, U10 HY6264AxP, U11 HY6264AxP, U12 2764, U13 2764, U14 2764, U15 2764, U16 74LS30, U17 74LS32, U18 74LS139, U19 74LS27, U2 8284, U3 74LS245, U4 74LS245, U5 74LS373, U6 74LS373, U7 74LS373, U8 HY6264AxP, U9 HY6264AxP, Y1 15MHz

Commit message: LE4 kicad v2
start of separating sheets
Parts:
- removed U16: 74LS30, symbol 74xx:74LS30
- removed U17: 74LS32, symbol 74xx:74LS32
- removed U18: 74LS139, symbol 74xx:74LS139
- removed U19: 74LS27, symbol 74xx:74LS27
- removed U3, U4: 74LS245, symbol 74xx:74LS245
- removed U5, U6, U7: 74LS373, symbol 74xx:74LS373
Connections:
- net ~{RD}: now also U12.22 (~{OE}), U13.22 (~{OE}), U14.22 (~{OE}), U15.22 (~{OE}); no longer U12.20 (~{CE}), U13.20 (~{CE}), U14.20 (~{CE}), U15.20 (~{CE})
- net ~{ROM1}: now also U12.20 (~{CE}), U13.20 (~{CE}); no longer U12.22 (~{OE}), U13.22 (~{OE})
- net ~{ROM2}: now also U14.20 (~{CE}), U15.20 (~{CE}); no longer U14.22 (~{OE}), U15.22 (~{OE})
- no-connect marks 14 -> 5
Other:
- added sheet Address Decoder (decoder.kicad_sch)
- added sheet Bus Buffering and Latching (bus.kicad_sch)
- added sheet RAM Array (ram.kicad_sch)
- added sheet ROM Array (rom.kicad_sch)
- moved on the sheet: C1, D1, R1, SW1, U1, U10, U11, U12, U13, U14, U15, U2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

Commit message: final updates to LE4-2
Parts:
- removed U10, U11, U8, U9: HY6264AxP, Package_DIP:DIP-28_W15.24mm, symbol Memory_RAM:HY6264AxP
- removed U12, U13, U14, U15: 2764, Package_DIP:DIP-28_W15.24mm, symbol Memory_EPROM:2764
- added J1: Jack-DC, symbol Connector:Jack-DC
- R1: value 10k -> 10kΩ
Connections:
- net GND: now also J1.2
- net VCC: now also J1.1
- net ALE renamed Bus Buffering and Latching/ALE
- net DT/~{R} renamed Bus Buffering and Latching/DT/~{R}
- net M/~{IO} renamed Address Decoder/M/~{IO}
- net ~{BHE}/S7 renamed Bus Buffering and Latching/~{BHE}/S7
- net ~{DEN} renamed Bus Buffering and Latching/~{DEN}
- net ~{RD} renamed RAM Array/~{RD}
- net ~{WR} renamed Address Decoder/~{WR}
Other:
- sheet Address Decoder ports: added A[0..19], M/~{IO}, ~{BHE}, ~{HWR}, ~{LWR}, ~{RAM[1..2]}, ~{ROM[1..2]}, ~{WR}; removed none
- sheet Bus Buffering and Latching ports: added AD[0..19], ALE, A[0..19], DT/~{R}, D[0..15], ~{BHE}, ~{BHE}/S7, ~{DEN}; removed none
- sheet RAM Array ports: added A[0..19], D[0..15], ~{HWR}, ~{LWR}, ~{RAM[1..2]}, ~{RD}; removed none
- sheet ROM Array ports: added A[0..19], D[0..15], ~{RD}, ~{ROM[1..2]}; removed none
- note added: "8284A to 8086 µP"
- note added: "Memory Interfacing"
- note removed: "RAM Set 1"
- note removed: "RAM Set 2"
- note removed: "ROM Set 1"
- note removed: "ROM Set 2"
- company: (none) -> Root Sheet
- title: (none) -> Team1_LE4-2: Memory Interfacing (with Addressing Decoding)
- moved on the sheet: C1, D1, R1, SW1, U1, U2, Y1
