File: LE4/Team1_LE4-2/bus.kicad_sch (KiCad schematic)
At the start: 5 parts, among them U3 74LS245, U4 74LS245, U5 74LS373, U6 74LS373, U7 74LS373

Commit message: final updates to LE4-2
Other:
- note added: "Address Bus Latching"
- note added: "Data Bus Buffering"
- company: (none) -> Bus Buffering and Latching sheet
- title: (none) -> Team1_LE4-2: Memory Interfacing (with Addressing Decoding)
- moved on the sheet: U3, U4, U5, U6, U7
