File: LE4/Team1_LE4-2/ram.kicad_sch (KiCad schematic)
At the start: 0 parts

Commit message: final updates to LE4-2
Parts:
- added U10, U11, U8, U9: HY6264AxP, Package_DIP:DIP-28_W15.24mm, symbol Memory_RAM:HY6264AxP
Connections:
- new net A1: U10.10 (A0), U11.10 (A0), U8.10 (A0), U9.10 (A0)
- new net A10: U10.24 (A9), U11.24 (A9), U8.24 (A9), U9.24 (A9)
- new net A11: U10.21 (A10), U11.21 (A10), U8.21 (A10), U9.21 (A10)
- new net A12: U10.23 (A11), U11.23 (A11), U8.23 (A11), U9.23 (A11)
- new net A13: U10.2 (A12), U11.2 (A12), U8.2 (A12), U9.2 (A12)
- new net A2: U10.9 (A1), U11.9 (A1), U8.9 (A1), U9.9 (A1)
- new net A3: U10.8 (A2), U11.8 (A2), U8.8 (A2), U9.8 (A2)
- new net A4: U10.7 (A3), U11.7 (A3), U8.7 (A3), U9.7 (A3)
- new net A5: U10.6 (A4), U11.6 (A4), U8.6 (A4), U9.6 (A4)
- new net A6: U10.5 (A5), U11.5 (A5), U8.5 (A5), U9.5 (A5)
- new net A7: U10.4 (A6), U11.4 (A6), U8.4 (A6), U9.4 (A6)
- new net A8: U10.3 (A7), U11.3 (A7), U8.3 (A7), U9.3 (A7)
- new net A9: U10.25 (A8), U11.25 (A8), U8.25 (A8), U9.25 (A8)
- new net D0: U11.11 (I/O0), U9.11 (I/O0)
- new net D1: U11.12 (I/O1), U9.12 (I/O1)
- new net D10: U10.13 (I/O2), U8.13 (I/O2)
- new net D11: U10.15 (I/O3), U8.15 (I/O3)
- new net D12: U10.16 (I/O4), U8.16 (I/O4)
- new net D13: U10.17 (I/O5), U8.17 (I/O5)
- new net D14: U10.18 (I/O6), U8.18 (I/O6)
- new net D15: U10.19 (I/O7), U8.19 (I/O7)
- new net D2: U11.13 (I/O2), U9.13 (I/O2)
- new net D3: U11.15 (I/O3), U9.15 (I/O3)
- new net D4: U11.16 (I/O4), U9.16 (I/O4)
- new net D5: U11.17 (I/O5), U9.17 (I/O5)
- new net D6: U11.18 (I/O6), U9.18 (I/O6)
- new net D7: U11.19 (I/O7), U9.19 (I/O7)
- new net D8: U10.11 (I/O0), U8.11 (I/O0)
- new net D9: U10.12 (I/O1), U8.12 (I/O1)
- new net GND: U10.14 (GND), U11.14 (GND), U8.14 (GND), U9.14 (GND)
- new net VCC: U10.26 (CS2), U10.28 (VCC), U11.26 (CS2), U11.28 (VCC), U8.26 (CS2), U8.28 (VCC), U9.26 (CS2), U9.28 (VCC)
- new net ~{HWR}: U10.27 (~{WE}), U11.27 (~{WE}), U8.27 (~{WE})
- new net ~{LWR}: U9.27 (~{WE})
- new net ~{RAM1}: U8.20 (~{CS1}), U9.20 (~{CS1})
- new net ~{RAM2}: U10.20 (~{CS1}), U11.20 (~{CS1})
- new net ~{RD}: U10.22 (~{OE}), U11.22 (~{OE}), U8.22 (~{OE}), U9.22 (~{OE})
Other:
- note added: "RAM Set 1"
- note added: "RAM Set 1 (High Bank)"
- note added: "RAM Set 1 (Low Bank)"
- note added: "RAM Set 2"
- note added: "RAM Set 2 (High Bank)"
- note added: "RAM Set 2 (Low Bank)"
- company: (none) -> RAM Array sheet
- title: (none) -> Team1_LE4-2: Memory Interfacing (with Addressing Decoding)
