File: LE4/Team1_LE4-2/rom.kicad_sch (KiCad schematic)
At the start: 0 parts

Commit message: final updates to LE4-2
Parts:
- added U12, U13, U14, U15: 2764, Package_DIP:DIP-28_W15.24mm, symbol Memory_EPROM:2764
Connections:
- new net A1: U12.10 (A0), U13.10 (A0), U14.10 (A0), U15.10 (A0)
- new net A10: U12.24 (A9), U13.24 (A9), U14.24 (A9), U15.24 (A9)
- new net A11: U12.21 (A10), U13.21 (A10), U14.21 (A10), U15.21 (A10)
- new net A12: U12.23 (A11), U13.23 (A11), U14.23 (A11), U15.23 (A11)
- new net A13: U12.2 (A12), U13.2 (A12), U14.2 (A12), U15.2 (A12)
- new net A2: U12.9 (A1), U13.9 (A1), U14.9 (A1), U15.9 (A1)
- new net A3: U12.8 (A2), U13.8 (A2), U14.8 (A2), U15.8 (A2)
- new net A4: U12.7 (A3), U13.7 (A3), U14.7 (A3), U15.7 (A3)
- new net A5: U12.6 (A4), U13.6 (A4), U14.6 (A4), U15.6 (A4)
- new net A6: U12.5 (A5), U13.5 (A5), U14.5 (A5), U15.5 (A5)
- new net A7: U12.4 (A6), U13.4 (A6), U14.4 (A6), U15.4 (A6)
- new net A8: U12.3 (A7), U13.3 (A7), U14.3 (A7), U15.3 (A7)
- new net A9: U12.25 (A8), U13.25 (A8), U14.25 (A8), U15.25 (A8)
- new net D0: U13.11 (D0), U15.11 (D0)
- new net D1: U13.12 (D1), U15.12 (D1)
- new net D10: U12.13 (D2), U14.13 (D2)
- new net D11: U12.15 (D3), U14.15 (D3)
- new net D12: U12.16 (D4), U14.16 (D4)
- new net D13: U12.17 (D5), U14.17 (D5)
- new net D14: U12.18 (D6), U14.18 (D6)
- new net D15: U12.19 (D7), U14.19 (D7)
- new net D2: U13.13 (D2), U15.13 (D2)
- new net D3: U13.15 (D3), U15.15 (D3)
- new net D4: U13.16 (D4), U15.16 (D4)
- new net D5: U13.17 (D5), U15.17 (D5)
- new net D6: U13.18 (D6), U15.18 (D6)
- new net D7: U13.19 (D7), U15.19 (D7)
- new net D8: U12.11 (D0), U14.11 (D0)
- new net D9: U12.12 (D1), U14.12 (D1)
- new net GND: U12.14 (GND), U13.14 (GND), U14.14 (GND), U15.14 (GND)
- new net VCC: U12.1 (VPP), U12.27 (~{PGM}), U12.28 (VCC), U13.1 (VPP), U13.27 (~{PGM}), U13.28 (VCC), U14.1 (VPP), U14.27 (~{PGM}), U14.28 (VCC), U15.1 (VPP), U15.27 (~{PGM}), U15.28 (VCC)
- new net ~{RD}: U12.22 (~{OE}), U13.22 (~{OE}), U14.22 (~{OE}), U15.22 (~{OE})
- new net ~{ROM1}: U12.20 (~{CE}), U13.20 (~{CE})
- new net ~{ROM2}: U14.20 (~{CE}), U15.20 (~{CE})
Other:
- note added: "ROM Set 1"
- note added: "ROM Set 1 (High Bank)"
- note added: "ROM Set 1 (Low Bank)"
- note added: "ROM Set 2"
- note added: "ROM Set 2 (High Bank)"
- note added: "ROM Set 2 (Low Bank)"
- company: (none) -> ROM Array sheet
- title: (none) -> Team1_LE4-2: Memory Interfacing (with Addressing Decoding)
